File: ReplicatorElectronics/rep_ctrlr/rep_ctrlr.sch (EAGLE design)
At the start: 98 parts, among them IC1 MICROCHIP_PIC32MX7X5F256L-PF, IC2 MICROCHIP_MCP6001-LT, IC3 MICROCHIP_MCP6001-LT, IC4 MICROCHIP_MCP6001-LT, IC5 MICROCHIP_MCP6001-LT, J1 ATX24RH, J10 SBH11-PBPC-D07-ST-BK, J11 SBH11-PBPC-D07-ST-BK, J12 SBH11-PBPC-D07-ST-BK, J13 SBH11-PBPC-D07-ST-BK, J14 SBH11-PBPC-D07-ST-BK, J15 SBH11-PBPC-D07-ST-BK, J16 SBH11-PBPC-D07-ST-BK, J17 SBH11-PBPC-D07-ST-BK, J18 SI-50170-F, J19 70553-0106, J4 RJ11-2L-B, J6 SBH11-PBPC-D05-ST-BK, J7 SBH11-PBPC-D05-ST-BK, J8 SBH11-PBPC-D05-ST-BK, J9 SBH11-PBPC-D05-ST-BK, Q1 ASFL1, Q2 ASFL1, U18 LDS3985XX33

Commit message: 5/14/12: Began power rail routing and display connector routing.
~ 2 hrs
Parts:
- U$1: value SBH11-PBPC-D13-ST-BK -> SBH11-PBPC-D17-ST-BK; device SBH11-PBPC-D13-ST-BK:SBH11-PBPC-D13-ST-BK -> SBH11-PBPC-D17-ST-BK:SBH11-PBPC-D17-ST-BK
Connections:
- removed net ETXERR: IC1PB.AN11/ERXERR/AETXERR/PMA12/RB11
- removed net PICCLKO: IC1PC.OSC2/CLKO/RC15
- net +3V3: now also C1.1, C18.1, C2.1, C3.1, C4.1, C5.1, C6.1, IC1MISC.VDD@1, IC1MISC.VDD@2, IC1MISC.VDD@3, IC1MISC.VDD@4, IC1MISC.VDD@5, IC1MISC.VDD@6, IC1MISC.VUSB, Q2.VCC, R1.2, R2.2
- net DGND: now also U$1.30, U$1.32; no longer U$1.22, U$1.24, U$1.26
- net HEAT0_ON: now also IC1PG.ECRS/SDA2A/SDI2A/U2ARX/PMA4/CN9/RG7
- net LCD_CS: now also U$1.22
- net LCD_RD: now also U$1.23
- net LCD_RST: now also U$1.25
- net LCD_WR: now also U$1.24
- net SD_CSN: now also U$1.26; no longer U$1.18
- net SD_SP_MISO: now also U$1.29; no longer U$1.20
- net SD_SP_MOSI: now also U$1.28; no longer U$1.21
- net SD_SP_SCK: now also U$1.27; no longer U$1.19
- net VCC: now also U$1.31, U$1.33; no longer C1.1, C18.1, C2.1, C3.1, C4.1, C5.1, C6.1, IC1MISC.VDD@1, IC1MISC.VDD@2, IC1MISC.VDD@3, IC1MISC.VDD@4, IC1MISC.VDD@5, IC1MISC.VDD@6, IC1MISC.VUSB, Q2.VCC, R1.2, R2.2, U$1.23, U$1.25
- net X+: now also U$1.18
- net X-: now also U$1.19
- net Y+: now also U$1.20
- net Y-: now also U$1.21

Commit message: 5/15/12: Completed power routing, completed servo connector routing save for PIC traces (which now lead nearby PIC but do not connect to pins). Heater connectors and PIC IO routing remain largely untouched. Some passives have yet to be placed.
~ 3 hrs.
Connections:
- net ENC_3_3V: now also J19.5, U$1.31, U$1.33
- net SERVO0: now also U$3.2A4; no longer J10.8, U$3.1A1
- net SERVO0_5V: now also J10.8, U$3.2Y4; no longer U$3.1Y1
- net SERVO1: now also U$3.1A1; no longer J11.8, U$3.1A2
- net SERVO1_5V: now also J11.8, U$3.1Y1; no longer U$3.1Y2
- net SERVO2: now also U$3.2A2; no longer J12.8, U$3.1A3
- net SERVO2_5V: now also J12.8, U$3.2Y2; no longer U$3.1Y3
- net SERVO3: now also U$3.2A1; no longer J13.8, U$3.1A4
- net SERVO3_5V: now also J13.8, U$3.2Y1; no longer U$3.1Y4
- net SERVO4: now also U$3.1A3; no longer J14.8, U$3.2A1
- net SERVO4_5V: now also J14.8, U$3.1Y3; no longer U$3.2Y1
- net SERVO5: now also U$3.2A3; no longer J15.8, U$3.2A2
- net SERVO5_5V: now also J15.8, U$3.2Y3; no longer U$3.2Y2
- net SERVO6: now also U$3.1A2; no longer J16.8, U$3.2A3
- net SERVO6_5V: now also J16.8, U$3.1Y2; no longer U$3.2Y3
- net SERVO7: now also U$3.1A4; no longer J17.8, U$3.2A4
- net SERVO7_5V: now also J17.8, U$3.1Y4; no longer U$3.2Y4
- net VCC: no longer J19.5, U$1.31, U$1.33

Commit message: 5/16/12: All but PHY-PIC signals, encoder SPI bus (PIC pins only), servo signals (3.3V side only), and temperature inputs routed.
~ 4 hrs.
Connections:
- net DB17: now also U$1.18; no longer U$1.17
- net ENC_3_3V: now also C19.1, Q1.VCC, R14.2, R15.2, R17.2, R18.2, R20.2, R21.2, R23.2, R24.2
- net VCC: no longer C19.1, Q1.VCC, R14.2, R15.2, R17.2, R18.2, R20.2, R21.2, R23.2, R24.2
- net X+: now also U$1.17; no longer U$1.18

Commit message: 5/19/12: 18 PIC connections left. Ground currently fractured.
~3 hrs spent between last commit and this one.
Parts:
- C10, C11, C12, C13, C14, C15, C16, C17, C18, C7, C8, C9: device resistor:C-USC0603 -> resistor:C-USC0402
- C19, C30: device rcl:C-USC0603 -> resistor:C-USC0402
- R1, R10, R13, R14, R15, R16, R17, R18, R19, R2, R20, R21, R22, R23, R24, R9: device resistor:R-US_R0603 -> resistor:R-US_R0402
Connections:
- net A0: now also U$1.24; no longer U$1.1
- net DB1: now also U$1.4; no longer U$1.3
- net DB2: now also U$1.3; no longer U$1.4
- net LCD_WR: now also U$1.1; no longer U$1.24

Commit message: 5/27/12: 5 PIC pins remain to be routed (3 encoder signals and encoder SPI MISO/MOSI), as well as buffers/passives around heater connectors. Cleanup will be required.
~ 6 hrs.
Parts:
- C1, C2, C3, C4, C5, C6: device resistor:C-USC0603 -> resistor:C-USC0402
Connections:
- net A0: now also U$1.23; no longer U$1.24
- net DB0: now also U$1.10; no longer U$1.2
- net DB1: now also U$1.9; no longer U$1.4
- net DB10: now also U$1.7; no longer U$1.10
- net DB11: now also U$1.8; no longer U$1.11
- net DB12: now also U$1.5; no longer U$1.12
- net DB13: now also U$1.6; no longer U$1.13
- net DB14: now also U$1.1; no longer U$1.14
- net DB15: now also U$1.2; no longer U$1.15
- net DB16: now also U$1.4; no longer U$1.16
- net DB17: now also U$1.3; no longer U$1.18
- net DB2: now also U$1.12; no longer U$1.3
- net DB3: now also U$1.11; no longer U$1.5
- net DB4: now also U$1.14; no longer U$1.6
- net DB5: now also U$1.13; no longer U$1.7
- net DB6: now also U$1.16; no longer U$1.8
- net DB7: now also U$1.15; no longer U$1.9
- net HEAT1_ON: now also IC1PB.AN4/C1IN-/CN6/RB4; no longer IC1PG.TRD1/RG12
- net HEAT3_ON: now also IC1PB.AN5/C1IN+/VBUSON/CN7/RB5; no longer IC1PG.TRD2/RG14
- net LCD_CS: now also U$1.19; no longer U$1.22
- net LCD_RD: now also U$1.17; no longer U$1.23
- net LCD_RST: now also U$1.20; no longer U$1.25
- net LCD_WR: now also U$1.18; no longer U$1.1
- net SD_CSN: now also U$1.24; no longer U$1.26
- net TEMP0_BUF: now also IC1PB.AN3/C2IN+/CN5/RB3; no longer IC1PB.PGED1/AN0/CN2/RB0
- net TEMP3_BUF: now also IC1PB.PGED1/AN0/CN2/RB0; no longer IC1PB.AN3/C2IN+/CN5/RB3
- net X+: now also IC1PG.TRD2/RG14, U$1.26; no longer IC1PB.AN4/C1IN-/CN6/RB4, U$1.17
- net X-: now also U$1.21; no longer U$1.19
- net Y+: now also IC1PG.TRD1/RG12, U$1.25; no longer IC1PB.AN5/C1IN+/VBUSON/CN7/RB5, U$1.20
- net Y-: now also U$1.22; no longer U$1.21

Commit message: 5/28/12: Preliminary placement and routing complete, need to clean up DRC errors.
~ 2 hrs.
Connections:
- net ENC2_CSN: now also IC1PB.AN13/ERXD1/AECOL/PMA10/RB13; no longer IC1PA.SCL2/RA2
- net ENC4_CSN: now also IC1PA.VREF-/CVREF-/AERXD2/PMA7/RA9; no longer IC1PA.TDI/RA4
- net ENC5_CSN: now also IC1PB.AN14/ERXD2/AETXD3/PMALH/PMA1/RB14; no longer IC1PA.TDO/RA5
Changed lines of the file:
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@@
 <net name="ENC2_CSN" class="0">
-<segment>
-<wire x1="-63.5" y1="-30.48" x2="-48.26" y2="-30.48" width="0.1524" layer="91"/>
-<label x="-60.96" y="-30.48" size="1.778" layer="95"/>
-<pinref part="IC1" gate="PA" pin="SCL2/RA2"/>
-</segment>
 <segment>
 <wire x1="622.3" y1="-149.86" x2="609.6" y2="-149.86" width="0.1524" layer="91"/>
 <label x="609.6" y="-149.86" size="1.778" layer="95"/>
 <pinref part="J12" gate="G$1" pin="7"/>
+</segment>
+<segment>
+<wire x1="-63.5" y1="-106.68" x2="-48.26" y2="-106.68" width="0.1524" layer="91"/>
+<label x="-60.96" y="-106.68" size="1.778" layer="95"/>
+<pinref part="IC1" gate="PB" pin="AN13/ERXD1/AECOL/PMA10/RB13"/>
 </segment>
 </net>
@@
 <net name="ENC4_CSN" class="0">
 <segment>
-<wire x1="-63.5" y1="-35.56" x2="-48.26" y2="-35.56" width="0.1524" layer="91"/>
-<label x="-60.96" y="-35.56" size="1.778" layer="95"/>
-<pinref part="IC1" gate="PA" pin="TDI/RA4"/>
+<wire x1="-63.5" y1="-45.72" x2="-48.26" y2="-45.72" width="0.1524" layer="91"/>
+<label x="-60.96" y="-45.72" size="1.778" layer="95"/>
+<pinref part="IC1" gate="PA" pin="VREF-/CVREF-/AERXD2/PMA7/RA9"/>
 </segment>
 <segment>
@@
 <net name="ENC5_CSN" class="0">
 <segment>
-<wire x1="-63.5" y1="-38.1" x2="-48.26" y2="-38.1" width="0.1524" layer="91"/>
-<label x="-60.96" y="-38.1" size="1.778" layer="95"/>
-<pinref part="IC1" gate="PA" pin="TDO/RA5"/>
-</segment>
-<segment>
 <wire x1="665.48" y1="-236.22" x2="652.78" y2="-236.22" width="0.1524" layer="91"/>
 <label x="652.78" y="-236.22" size="1.778" layer="95"/>
 <pinref part="J15" gate="G$1" pin="7"/>
 </segment>
+<segment>
+<wire x1="-63.5" y1="-109.22" x2="-48.26" y2="-109.22" width="0.1524" layer="91"/>
+<label x="-60.96" y="-109.22" size="1.778" layer="95"/>
+<pinref part="IC1" gate="PB" pin="AN14/ERXD2/AETXD3/PMALH/PMA1/RB14"/>
+</segment>
 </net>

Commit message: 5/30/12: Preliminary layout finished! Ready for review by Alex.
~ 2 hrs.
Parts:
- added C20: 0.1u, resistor:C-USC0402
- J4: value RJ11-2L-B -> (none); device con-tycoelectronics:RJ11-2L-B -> con-molex:22-23-2061
Connections:
- removed net VCC: J4.2
- net +3V3: now also J4-2.S
- net 5V_USB: now also C20.1
- net DGND: now also C20.2, J4-3.S; no longer J4.3
- net MCLRN: now also J4-1.S; no longer J4.1
- net PGEC: now also J4-5.S; no longer J4.5
- net PGED: now also J4-4.S; no longer J4.4
Changed lines of the file:
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@@
 <part name="J16" library="SBH11-PBPC-D07-ST-BK" deviceset="SBH11-PBPC-D07-ST-BK" device=""/>
 <part name="J17" library="SBH11-PBPC-D07-ST-BK" deviceset="SBH11-PBPC-D07-ST-BK" device=""/>
-<part name="J4" library="con-tycoelectronics" deviceset="RJ11" device="" technology="-2L-B"/>
-<part name="P+20" library="supply1" deviceset="VCC" device=""/>
 <part name="SUPPLY44" library="supply2" deviceset="DGND" device=""/>
 <part name="J19" library="70553-0109" deviceset="70553-0106" device=""/>
@@
 <part name="SUPPLY45" library="supply2" deviceset="DGND" device=""/>
 <part name="U$1" library="SBH11-PBPC-D17-ST-BK" deviceset="SBH11-PBPC-D17-ST-BK" device=""/>
+<part name="C20" library="resistor" deviceset="C-US" device="C0402" value="0.1u"/>
+<part name="SUPPLY46" library="supply2" deviceset="DGND" device=""/>
+<part name="J4" library="con-molex" deviceset="22-23-2061" device=""/>
 </parts>
 <sheets>
@@
 <instance part="J16" gate="G$1" x="782.32" y="-238.76"/>
 <instance part="J17" gate="G$1" x="886.46" y="-241.3"/>
-<instance part="J4" gate="G$1" x="88.9" y="-226.06"/>
-<instance part="P+20" gate="VCC" x="63.5" y="-218.44"/>
 <instance part="SUPPLY44" gate="G$1" x="63.5" y="-228.6"/>
 <instance part="J19" gate="G$1" x="139.7" y="-241.3"/>
@@
 <attribute name="NAME" x="287.02" y="-25.4" size="1.778" layer="94"/>
 </instance>
+<instance part="C20" gate="G$1" x="533.4" y="-104.14"/>
+<instance part="SUPPLY46" gate="G$1" x="533.4" y="-111.76"/>
+<instance part="J4" gate="-1" x="88.9" y="-220.98"/>
+<instance part="J4" gate="-2" x="88.9" y="-223.52"/>
+<instance part="J4" gate="-3" x="88.9" y="-226.06"/>
+<instance part="J4" gate="-4" x="88.9" y="-228.6"/>
+<instance part="J4" gate="-5" x="88.9" y="-231.14"/>
+<instance part="J4" gate="-6" x="88.9" y="-233.68"/>
 </instances>
 <busses>
 </busses>
 <nets>
-<net name="VCC" class="0">
-<segment>
-<pinref part="J4" gate="G$1" pin="2"/>
-<wire x1="86.36" y1="-223.52" x2="63.5" y2="-223.52" width="0.1524" layer="91"/>
-<pinref part="P+20" gate="VCC" pin="VCC"/>
-<wire x1="63.5" y1="-223.52" x2="63.5" y2="-220.98" width="0.1524" layer="91"/>
-</segment>
-</net>
 <net name="GND" class="0">
 <segment>
@@
 </segment>
 <segment>
-<pinref part="J4" gate="G$1" pin="1"/>
 <wire x1="86.36" y1="-220.98" x2="71.12" y2="-220.98" width="0.1524" layer="91"/>
 <label x="76.2" y="-220.98" size="1.778" layer="95"/>
+<pinref part="J4" gate="-1" pin="S"/>
 </segment>
 </net>
@@
 <pinref part="U$3" gate="G$1" pin="VCC"/>
 <wire x1="533.4" y1="-119.38" x2="546.1" y2="-119.38" width="0.1524" layer="91"/>
-<wire x1="546.1" y1="-119.38" x2="546.1" y2="-109.22" width="0.1524" layer="91"/>
+<wire x1="546.1" y1="-119.38" x2="546.1" y2="-111.76" width="0.1524" layer="91"/>
 <label x="543.56" y="-109.22" size="1.778" layer="95"/>
+<pinref part="C20" gate="G$1" pin="1"/>
+<wire x1="546.1" y1="-111.76" x2="546.1" y2="-109.22" width="0.1524" layer="91"/>
+<wire x1="533.4" y1="-101.6" x2="533.4" y2="-93.98" width="0.1524" layer="91"/>
+<wire x1="533.4" y1="-93.98" x2="541.02" y2="-93.98" width="0.1524" layer="91"/>
+<wire x1="541.02" y1="-93.98" x2="541.02" y2="-111.76" width="0.1524" layer="91"/>
+<wire x1="541.02" y1="-111.76" x2="546.1" y2="-111.76" width="0.1524" layer="91"/>
+<junction x="546.1" y="-111.76"/>
 </segment>
 </net>
@@
 </segment>
 <segment>
-<pinref part="J4" gate="G$1" pin="3"/>
 <wire x1="86.36" y1="-226.06" x2="63.5" y2="-226.06" width="0.1524" layer="91"/>
 <pinref part="SUPPLY44" gate="G$1" pin="DGND"/>
+<pinref part="J4" gate="-3" pin="S"/>
 </segment>
 <segment>
@@
 <junction x="337.82" y="-106.68"/>
 </segment>
+<segment>
+<pinref part="C20" gate="G$1" pin="2"/>
+<pinref part="SUPPLY46" gate="G$1" pin="DGND"/>
+</segment>
 </net>
 <net name="DB0" class="0">
@@
 </segment>
 <segment>
-<pinref part="J4" gate="G$1" pin="5"/>
 <wire x1="86.36" y1="-231.14" x2="71.12" y2="-231.14" width="0.1524" layer="91"/>
 <label x="76.2" y="-231.14" size="1.778" layer="95"/>
+<pinref part="J4" gate="-5" pin="S"/>
 </segment>
 </net>
@@
 <wire x1="86.36" y1="-228.6" x2="71.12" y2="-228.6" width="0.1524" layer="91"/>
 <label x="71.12" y="-228.6" size="1.778" layer="95"/>
-<pinref part="J4" gate="G$1" pin="4"/>
+<pinref part="J4" gate="-4" pin="S"/>
 </segment>
 </net>
@@
 <label x="-116.84" y="-167.64" size="1.778" layer="95"/>
 </segment>
-</net>
+<segment>
+<wire x1="86.36" y1="-223.52" x2="63.5" y2="-223.52" width="0.1524" layer="91"/>
+<wire x1="63.5" y1="-223.52" x2="63.5" y2="-220.98" width="0.1524" layer="91"/>
+<pinref part="J4" gate="-2" pin="S"/>
+</segment>
+</net>

Commit message: 5/3/12: Minor cleanup.
~ 0.5 hr.
Parts:
- renumbered U$1 to J20
Changed lines of the file:
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@@
 <part name="SUPPLY37" library="supply2" deviceset="DGND" device=""/>
 <part name="SUPPLY45" library="supply2" deviceset="DGND" device=""/>
-<part name="U$1" library="SBH11-PBPC-D17-ST-BK" deviceset="SBH11-PBPC-D17-ST-BK" device=""/>
+<part name="J20" library="SBH11-PBPC-D17-ST-BK" deviceset="SBH11-PBPC-D17-ST-BK" device=""/>
 <part name="C20" library="resistor" deviceset="C-US" device="C0402" value="0.1u"/>
 <part name="SUPPLY46" library="supply2" deviceset="DGND" device=""/>
@@
 <instance part="SUPPLY37" gate="G$1" x="472.44" y="-127"/>
 <instance part="SUPPLY45" gate="G$1" x="474.98" y="-172.72"/>
-<instance part="U$1" gate="G$1" x="289.56" y="-66.04" smashed="yes">
+<instance part="J20" gate="G$1" x="289.56" y="-66.04" smashed="yes">
 <attribute name="NAME" x="287.02" y="-25.4" size="1.778" layer="94"/>
 </instance>
@@
 </segment>
 <segment>
-<pinref part="U$1" gate="G$1" pin="24"/>
+<pinref part="J20" gate="G$1" pin="24"/>
 <wire x1="304.8" y1="-86.36" x2="332.74" y2="-86.36" width="0.1524" layer="91"/>
 <label x="309.88" y="-86.36" size="1.778" layer="95"/>
@@
 <segment>
 <pinref part="SUPPLY2" gate="G$1" pin="DGND"/>
-<pinref part="U$1" gate="G$1" pin="32"/>
+<pinref part="J20" gate="G$1" pin="32"/>
 <wire x1="304.8" y1="-106.68" x2="337.82" y2="-106.68" width="0.1524" layer="91"/>
 <wire x1="337.82" y1="-106.68" x2="337.82" y2="-116.84" width="0.1524" layer="91"/>
-<pinref part="U$1" gate="G$1" pin="30"/>
+<pinref part="J20" gate="G$1" pin="30"/>
 <wire x1="304.8" y1="-101.6" x2="337.82" y2="-101.6" width="0.1524" layer="91"/>
 <wire x1="337.82" y1="-101.6" x2="337.82" y2="-106.68" width="0.1524" layer="91"/>
@@
 <wire x1="304.8" y1="-50.8" x2="332.74" y2="-50.8" width="0.1524" layer="91"/>
 <label x="309.88" y="-50.8" size="1.778" layer="95"/>
-<pinref part="U$1" gate="G$1" pin="10"/>
+<pinref part="J20" gate="G$1" pin="10"/>
 </segment>
 </net>
@@
 <wire x1="276.86" y1="-50.8" x2="248.92" y2="-50.8" width="0.1524" layer="91"/>
 <label x="256.54" y="-50.8" size="1.778" layer="95"/>
-<pinref part="U$1" gate="G$1" pin="9"/>
+<pinref part="J20" gate="G$1" pin="9"/>
 </segment>
 </net>
@@
 <wire x1="304.8" y1="-55.88" x2="332.74" y2="-55.88" width="0.1524" layer="91"/>
 <label x="309.88" y="-55.88" size="1.778" layer="95"/>
-<pinref part="U$1" gate="G$1" pin="12"/>
+<pinref part="J20" gate="G$1" pin="12"/>
 </segment>
 </net>
@@
 <wire x1="276.86" y1="-55.88" x2="248.92" y2="-55.88" width="0.1524" layer="91"/>
 <label x="256.54" y="-55.88" size="1.778" layer="95"/>
-<pinref part="U$1" gate="G$1" pin="11"/>
+<pinref part="J20" gate="G$1" pin="11"/>
 </segment>
 </net>
@@
 <wire x1="276.86" y1="-45.72" x2="248.92" y2="-45.72" width="0.1524" layer="91"/>
 <label x="256.54" y="-45.72" size="1.778" layer="95"/>
-<pinref part="U$1" gate="G$1" pin="7"/>
+<pinref part="J20" gate="G$1" pin="7"/>
 </segment>
 </net>
@@
 <wire x1="304.8" y1="-45.72" x2="332.74" y2="-45.72" width="0.1524" layer="91"/>
 <label x="309.88" y="-45.72" size="1.778" layer="95"/>
-<pinref part="U$1" gate="G$1" pin="8"/>
+<pinref part="J20" gate="G$1" pin="8"/>
 </segment>
 </net>
@@
 <wire x1="304.8" y1="-60.96" x2="332.74" y2="-60.96" width="0.1524" layer="91"/>
 <label x="309.88" y="-60.96" size="1.778" layer="95"/>
-<pinref part="U$1" gate="G$1" pin="14"/>
+<pinref part="J20" gate="G$1" pin="14"/>
 </segment>
 </net>
@@
 <wire x1="304.8" y1="-40.64" x2="332.74" y2="-40.64" width="0.1524" layer="91"/>
 <label x="309.88" y="-40.64" size="1.778" layer="95"/>
-<pinref part="U$1" gate="G$1" pin="6"/>
+<pinref part="J20" gate="G$1" pin="6"/>
 </segment>
 </net>
@@
 <wire x1="304.8" y1="-35.56" x2="332.74" y2="-35.56" width="0.1524" layer="91"/>
 <label x="309.88" y="-35.56" size="1.778" layer="95"/>
-<pinref part="U$1" gate="G$1" pin="4"/>
+<pinref part="J20" gate="G$1" pin="4"/>
 </segment>
 </net>
@@
 <wire x1="276.86" y1="-35.56" x2="248.92" y2="-35.56" width="0.1524" layer="91"/>
 <label x="256.54" y="-35.56" size="1.778" layer="95"/>
-<pinref part="U$1" gate="G$1" pin="3"/>
+<pinref part="J20" gate="G$1" pin="3"/>
 </segment>
 </net>
@@
 <wire x1="276.86" y1="-60.96" x2="248.92" y2="-60.96" width="0.1524" layer="91"/>
 <label x="256.54" y="-60.96" size="1.778" layer="95"/>
-<pinref part="U$1" gate="G$1" pin="13"/>
+<pinref part="J20" gate="G$1" pin="13"/>
 </segment>
 </net>
@@
 <wire x1="304.8" y1="-66.04" x2="332.74" y2="-66.04" width="0.1524" layer="91"/>
 <label x="309.88" y="-66.04" size="1.778" layer="95"/>
-<pinref part="U$1" gate="G$1" pin="16"/>
+<pinref part="J20" gate="G$1" pin="16"/>
 </segment>
 </net>
@@
 <wire x1="276.86" y1="-66.04" x2="248.92" y2="-66.04" width="0.1524" layer="91"/>
 <label x="256.54" y="-66.04" size="1.778" layer="95"/>
-<pinref part="U$1" gate="G$1" pin="15"/>
+<pinref part="J20" gate="G$1" pin="15"/>
 </segment>
 </net>
 <net name="X+" class="0">
 <segment>
-<pinref part="U$1" gate="G$1" pin="26"/>
+<pinref part="J20" gate="G$1" pin="26"/>
 <wire x1="304.8" y1="-91.44" x2="332.74" y2="-91.44" width="0.1524" layer="91"/>
 <label x="309.88" y="-91.44" size="1.778" layer="95"/>
@@
 <net name="Y+" class="0">
 <segment>
-<pinref part="U$1" gate="G$1" pin="25"/>
+<pinref part="J20" gate="G$1" pin="25"/>
 <wire x1="276.86" y1="-91.44" x2="248.92" y2="-91.44" width="0.1524" layer="91"/>
 <label x="256.54" y="-91.44" size="1.778" layer="95"/>
@@
 <wire x1="276.86" y1="-81.28" x2="248.92" y2="-81.28" width="0.1524" layer="91"/>
 <label x="256.54" y="-81.28" size="1.778" layer="95"/>
-<pinref part="U$1" gate="G$1" pin="21"/>
+<pinref part="J20" gate="G$1" pin="21"/>
 </segment>
 </net>
@@
 </segment>
 <segment>
-<pinref part="U$1" gate="G$1" pin="22"/>
+<pinref part="J20" gate="G$1" pin="22"/>
 <wire x1="304.8" y1="-81.28" x2="332.74" y2="-81.28" width="0.1524" layer="91"/>
 <label x="309.88" y="-81.28" size="1.778" layer="95"/>
@@
 </segment>
 <segment>
-<pinref part="U$1" gate="G$1" pin="23"/>
+<pinref part="J20" gate="G$1" pin="23"/>
 <wire x1="276.86" y1="-86.36" x2="248.92" y2="-86.36" width="0.1524" layer="91"/>
 <label x="256.54" y="-86.36" size="1.778" layer="95"/>
@@
 <wire x1="276.86" y1="-76.2" x2="248.92" y2="-76.2" width="0.1524" layer="91"/>
 <label x="256.54" y="-76.2" size="1.778" layer="95"/>
-<pinref part="U$1" gate="G$1" pin="19"/>
+<pinref part="J20" gate="G$1" pin="19"/>
 </segment>
 </net>
@@
 <wire x1="304.8" y1="-71.12" x2="332.74" y2="-71.12" width="0.1524" layer="91"/>
 <label x="309.88" y="-71.12" size="1.778" layer="95"/>
-<pinref part="U$1" gate="G$1" pin="18"/>
+<pinref part="J20" gate="G$1" pin="18"/>
 </segment>
 </net>
@@
 <wire x1="276.86" y1="-71.12" x2="248.92" y2="-71.12" width="0.1524" layer="91"/>
 <label x="256.54" y="-71.12" size="1.778" layer="95"/>
-<pinref part="U$1" gate="G$1" pin="17"/>
+<pinref part="J20" gate="G$1" pin="17"/>
 </segment>
 </net>
@@
 <wire x1="304.8" y1="-76.2" x2="332.74" y2="-76.2" width="0.1524" layer="91"/>
 <label x="309.88" y="-76.2" size="1.778" layer="95"/>
-<pinref part="U$1" gate="G$1" pin="20"/>
+<pinref part="J20" gate="G$1" pin="20"/>
 </segment>
 </net>
@@
 <segment>
 <wire x1="241.3" y1="-104.14" x2="241.3" y2="-106.68" width="0.1524" layer="91"/>
-<pinref part="U$1" gate="G$1" pin="33"/>
+<pinref part="J20" gate="G$1" pin="33"/>
 <wire x1="276.86" y1="-111.76" x2="241.3" y2="-111.76" width="0.1524" layer="91"/>
-<pinref part="U$1" gate="G$1" pin="31"/>
+<pinref part="J20" gate="G$1" pin="31"/>
 <wire x1="276.86" y1="-106.68" x2="241.3" y2="-106.68" width="0.1524" layer="91"/>
 <wire x1="241.3" y1="-106.68" x2="241.3" y2="-111.76" width="0.1524" layer="91"/>
@@
 </segment>
 <segment>
-<pinref part="U$1" gate="G$1" pin="29"/>
+<pinref part="J20" gate="G$1" pin="29"/>
 <wire x1="276.86" y1="-101.6" x2="248.92" y2="-101.6" width="0.1524" layer="91"/>
 <label x="256.54" y="-101.6" size="1.778" layer="95"/>
@@
 </segment>
 <segment>
-<pinref part="U$1" gate="G$1" pin="28"/>
+<pinref part="J20" gate="G$1" pin="28"/>
 <wire x1="304.8" y1="-96.52" x2="332.74" y2="-96.52" width="0.1524" layer="91"/>
 <label x="309.88" y="-96.52" size="1.778" layer="95"/>
@@
 </segment>
 <segment>
-<pinref part="U$1" gate="G$1" pin="27"/>
+<pinref part="J20" gate="G$1" pin="27"/>
 <wire x1="276.86" y1="-96.52" x2="248.92" y2="-96.52" width="0.1524" layer="91"/>
 <label x="256.54" y="-96.52" size="1.778" layer="95"/>
@@
 <wire x1="276.86" y1="-30.48" x2="248.92" y2="-30.48" width="0.1524" layer="91"/>
 <label x="256.54" y="-30.48" size="1.778" layer="95"/>
-<pinref part="U$1" gate="G$1" pin="1"/>
+<pinref part="J20" gate="G$1" pin="1"/>
 </segment>
 </net>
@@
 <wire x1="304.8" y1="-30.48" x2="332.74" y2="-30.48" width="0.1524" layer="91"/>
 <label x="309.88" y="-30.48" size="1.778" layer="95"/>
-<pinref part="U$1" gate="G$1" pin="2"/>
+<pinref part="J20" gate="G$1" pin="2"/>
 </segment>
 </net>
@@
 <wire x1="276.86" y1="-40.64" x2="248.92" y2="-40.64" width="0.1524" layer="91"/>
 <label x="256.54" y="-40.64" size="1.778" layer="95"/>
-<pinref part="U$1" gate="G$1" pin="5"/>
-</segment>
-</net>
+<pinref part="J20" gate="G$1" pin="5"/>
+</segment>
+</net>
