File: ReplicatorElectronics/rep_ctrlr/rep_ctrlr.sch (EAGLE design)
At the start: 99 parts, among them IC1 MICROCHIP_PIC32MX7X5F256L-PF, IC2 MICROCHIP_MCP6001-LT, IC3 MICROCHIP_MCP6001-LT, IC4 MICROCHIP_MCP6001-LT, IC5 MICROCHIP_MCP6001-LT, J1 ATX24RH, J10 SBH11-PBPC-D07-ST-BK, J11 SBH11-PBPC-D07-ST-BK, J12 SBH11-PBPC-D07-ST-BK, J13 SBH11-PBPC-D07-ST-BK, J14 SBH11-PBPC-D07-ST-BK, J15 SBH11-PBPC-D07-ST-BK, J16 SBH11-PBPC-D07-ST-BK, J17 SBH11-PBPC-D07-ST-BK, J18 SI-50170-F, J19 70553-0106, J20 SBH11-PBPC-D17-ST-BK, J6 SBH11-PBPC-D05-ST-BK, J7 SBH11-PBPC-D05-ST-BK, J8 SBH11-PBPC-D05-ST-BK, J9 SBH11-PBPC-D05-ST-BK, Q1 ASFL1, Q2 ASFL1, U18 LDS3985XX33

Commit message: 5/8/12: Resolved refdes discrepancies, replaced unavailable components.
~ 1 hr.
Parts:
- removed C31, C32: 4.7uF, rcl:CPOL-USR/2012-12R
- removed C33: .1uF, rcl:C-USC0402
- removed J19: 70553-0106, 70553-0109:70553-0106
- removed R38, R39, R40: 49.9, resistor:R-US_R0603
- removed R41, R42: 270, resistor:R-US_R0603
- removed R44, R45: 10k, resistor:R-US_R0603
- removed R46: 10k, rcl:R-US_R0402
- added B1: FERRITE, resistor:R-US_R0805
- added C21: 0.1uF, resistor:C-USC0402
- added C22: 10u, resistor:C-USC0603
- added C23: 0.1uF, resistor:C-USC0603
- added J5: SBH11-PBPC-D05-ST-BK, SBH11-PBPC-D05-ST-BK:SBH11-PBPC-D05-ST-BK
- added R11, R12, R7: 10, resistor:R-US_R0402
- added R3, R4, R5, R6: 10K, resistor:R-US_R0402
- C27: value 0.1uF -> 1uF
- C29: value 1uF -> 4.7uF; device resistor:C-USC0603 -> rcl:CPOL-USR/2012-12R
- C30: value 0.1uF -> 4.7uF; device resistor:C-USC0402 -> rcl:CPOL-USR/2012-12R
- C8: value 10u -> .1uF; device resistor:C-USC0402 -> rcl:C-USC0402
- J1: value ATX24RH -> 0874272402
- J17: value SBH11-PBPC-D07-ST-BK -> SI-50170-F; device SBH11-PBPC-D07-ST-BK:SBH11-PBPC-D07-ST-BK -> con-stewart:SI-50170
- J18: value SI-50170-F -> 70553-0106; device con-stewart:SI-50170 -> 70553-0109:70553-0106
- J9: value SBH11-PBPC-D05-ST-BK -> SBH11-PBPC-D07-ST-BK; device SBH11-PBPC-D05-ST-BK:SBH11-PBPC-D05-ST-BK -> SBH11-PBPC-D07-ST-BK:SBH11-PBPC-D07-ST-BK
- R13, R16: value 10K -> 10
- R18, R20, R21, R23, R24: value 10 -> 49.9; device resistor:R-US_R0402 -> resistor:R-US_R0603
- R19, R22: value 10K -> 49.9; device resistor:R-US_R0402 -> resistor:R-US_R0603
- R2: value 10 -> 10k; device resistor:R-US_R0402 -> rcl:R-US_R0402
- R25, R26, R27, R28, R29, R30, R31, R32: value 50 -> 49.9
- R33: value 50 -> 12.1k 1%
- R34, R35: value 50 -> 270
- R36: value 12.1k 1% -> 10k
- R37: value 49.9 -> 10k
- R8: value FERRITE -> 10; device resistor:R-US_R0805 -> resistor:R-US_R0402
- renumbered IC1 to U1, IC2 to U5, IC3 to U7, IC4 to U4, IC5 to U6, J20 to J3, Q1 to X1, Q2 to X2, R43 to B2, U$2 to U2, U$3 to U8, U18 to U3
Connections:
- net +3V3: now also C29.+, R7.2; no longer C31.+, R2.2
- net 12V_HEAT: now also J5.1, J5.3, J5.5; no longer J9.1, J9.3, J9.5
- net 5V_SERVO: now also J9.1, J9.3, J9.5; no longer J17.1, J17.3, J17.5
- net 5V_USB: now also C30.+, R2.1; no longer C32.+, R46.1
- net DGND: now also B1.1, C21.2, C22.2, C23.2, C28.1, C29.-, C30.-, J17.C_GND, J17.S1, J17.S2, J18.6, J9.10, J9.12, R3.1, R33.1, R34.1, R35.1, R37.1, R4.1, R5.1, R6.1; no longer C28.2, C29.1, C30.2, C31.-, C32.-, C33.2, J17.10, J17.12, J18.C_GND, J18.S1, J18.S2, J19.6, R13.1, R16.1, R19.1, R22.1, R41.1, R42.1, R44.1, R45.1, R8.1
- net ECRSDV: now also R25.1; no longer R31.1
- net EMDC: now also R28.1; no longer R34.1
- net EMDIO: now also R27.1; no longer R33.1
- net ENC7_CSN: now also J9.7; no longer J17.7
- net ENC_3_3V: now also C23.1, J18.5, J9.14, R10.2, R11.2, R12.2, R13.2, R16.2; no longer C25.1, J17.14, J19.5, R18.2, R20.2, R21.2, R23.2, R24.2
- net ENC_MISO: now also J9.13; no longer J17.13
- net ENC_MOSI: now also J9.11; no longer J17.11
- net ENC_SCK: now also J9.9; no longer J17.9
- net EREFCLK: now also R26.1; no longer R32.1
- net ERXD0: now also R23.1; no longer R29.1
- net ERXD1: now also R22.1; no longer R28.1
- net ERXERR: now also R24.1; no longer R30.1
- net ETH_3_3V: now also C25.1, J17.RCT, J17.TCT, R18.2, R30.2, R31.2, R32.2; no longer C28.1, J18.RCT, J18.TCT, R37.2, R38.2, R39.2, R40.2
- net ETXD0: now also R20.1; no longer R26.1
- net ETXD1: now also R19.1; no longer R25.1
- net ETXEN: now also R21.1; no longer R27.1
- net GND: now also B1.2, J5.2, J5.4, J5.6, J5.8; no longer J17.2, J17.4, J17.6, J9.8, R8.2
- net HEAT3_ON: now also J5.7; no longer J9.7
- net LED1: now also J17.A; no longer J18.A
- net LED2: now also J17.A1, R36.2; no longer J18.A1, R45.2
- net N$1: now also R8.2; no longer R9.2
- net N$11: now also J5.9, R5.2; no longer J9.9, R16.2
- net N$12: now also J5.10, R15.1; no longer J9.10, R17.1
- net N$13: now also R11.1; no longer R14.1
- net N$14: now also R12.1; no longer R15.1
- net N$15: now also R16.1; no longer R18.1
- net N$16: now also R4.2; no longer R19.2
- net N$17: now also R13.1; no longer R20.1
- net N$18: now also R14.1; no longer R21.1
- net N$19: now also R6.2; no longer R22.2
- net N$2: now also R7.1; no longer R2.1
- net N$20: now also R17.1; no longer R23.1
- net N$21: now also R10.1; no longer R24.1
- net N$23: now also R19.2; no longer R25.2
- net N$24: now also R20.2; no longer R26.2
- net N$25: now also R21.2; no longer R27.2
- net N$26: now also R22.2; no longer R28.2
- net N$27: now also R23.2; no longer R29.2
- net N$28: now also R24.2; no longer R30.2
- net N$29: now also R25.2; no longer R31.2
- net N$30: now also R26.2; no longer R32.2
- net N$31: now also R27.2; no longer R33.2
- net N$32: now also R28.2; no longer R34.2
- net N$33: now also R29.2, R37.2; no longer R35.2, R44.2
- net N$34: now also J17.TD+, R30.1; no longer J18.TD+, R37.1
- net N$35: now also J17.TD-, R31.1; no longer J18.TD-, R38.1
- net N$36: now also J17.RD+, R32.1; no longer J18.RD+, R39.1
- net N$37: now also J17.RD-, R18.1; no longer J18.RD-, R40.1
- net N$38: now also R9.1; no longer R10.1
- net N$4: now also R9.2; no longer R10.2
- net N$40: now also R2.2; no longer R46.2
- net N$41: now also C8.1; no longer C33.1
- net N$42: now also J17.C, R35.2; no longer J18.C, R42.2
- net N$43: now also J17.C1, R34.2; no longer J18.C1, R41.2
- net N$44: now also C28.2; no longer C29.2
- net N$5: now also C22.1; no longer C8.1
- net N$52: now also R33.2; no longer R36.2
- net N$9: now also R3.2; no longer R13.2
- net NRST: now also R29.1; no longer R35.1
- net PICCLKI: now also R8.1; no longer R9.1
- net SD_SP_MISO: now also J18.3; no longer J19.3
- net SD_SP_MOSI: now also J18.4; no longer J19.4
- net SD_SP_SCK: now also J18.1; no longer J19.1
- net SERVO7_5V: now also J9.8; no longer J17.8
- net SP_CSN: now also J18.2; no longer J19.2
Other:
- moved on the sheet: C25, C26, C27, C28, C8, R10, R13, R14, R15, R16, R17, R18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
