File: electronics/ReplicatorElectronics/rep_ctrlr/Controller Rev 3.brd (EAGLE design)
At the start: 70 x 70 mm, 81 parts, among them IC2 MICROCHIP_MCP6001-LT, IC3 MICROCHIP_MCP6001-LT, IC4 MICROCHIP_MCP6001-LT, J1 ATX24RH, J10 WASP7PIN, J16 OSTVN04A150, J2 OSTVN04A150, J3 OSTVN04A150, Q1 DISCRETE_MMBT3904LT1G, Q11 DISCRETE_MMBT3904LT1G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

Commit message: Added values for heater section to the overlay
Parts:
- C2, C3: value .1uF -> 18p
Other:
- board text added: "10k"
- board text added: "3.3vreg"
- board text added: "330"
- board text added: "8mhz xtal"
- board text added: "Diode"
- board text added: "Ignore"
- board text added: "PIC32"
- board text added: "PNP"
- board text added: "SN74ACT244"
- board text added: "SWITCH"
- board text added: "Short me"
- board text added: "amp"
- board text added: "npn"
- board text added: "rgb"
